File: kicad_btkb/bt_keybrd.sch (KiCad schematic (older format))
At the start: 2 parts, among them IC1 MEGA32-A

Commit message: okay
Parts:
- added P? (x2): CONN_20, symbol CONN_20
- added P?: CONN_3X2, symbol CONN_3X2
Other:
- moved on the sheet: IC1, rn1
Changed lines of the file:
@@
 L MEGA32-A IC1
 U 1 1 538B7F7D
-P 3750 3700
-F 0 "IC1" H 3150 5530 50  0000 L BNN
-F 1 "MEGA32-A" H 3150 1800 50  0000 L BNN
-F 2 "avr-TQFP44" H 3750 3850 50  0001 C CNN
-F 3 "" H 3750 3700 60  0000 C CNN
-	1    3750 3700
+P 2200 3350
+F 0 "IC1" H 1600 5180 50  0000 L BNN
+F 1 "MEGA32-A" H 1600 1450 50  0000 L BNN
+F 2 "avr-TQFP44" H 2200 3500 50  0001 C CNN
+F 3 "" H 2200 3350 60  0000 C CNN
+	1    2200 3350
 	1    0    0    -1
 $EndComp
@@
 L rn-42 rn1
 U 1 1 538B85D8
-P 9300 2100
-F 0 "rn1" H 9300 2350 60  0000 C CNN
-F 1 "rn-42" H 9300 1150 60  0000 C CNN
-F 2 "" H 9250 2100 60  0000 C CNN
-F 3 "" H 9250 2100 60  0000 C CNN
-	1    9300 2100
+P 6850 8550
+F 0 "rn1" H 6850 8800 60  0000 C CNN
+F 1 "rn-42" H 6850 7600 60  0000 C CNN
+F 2 "" H 6800 8550 60  0000 C CNN
+F 3 "" H 6800 8550 60  0000 C CNN
+	1    6850 8550
 	1    0    0    -1
 $EndComp
+$Comp
+L CONN_20 P?
+U 1 1 538BD800
+P 2550 6950
+F 0 "P?" V 2500 6950 60  0000 C CNN
+F 1 "CONN_20" V 2600 6950 60  0000 C CNN
+F 2 "" H 2550 6950 60  0000 C CNN
+F 3 "" H 2550 6950 60  0000 C CNN
+	1    2550 6950
+	1    0    0    -1
+$EndComp
+$Comp
+L CONN_20 P?
+U 1 1 538BD861
+P 2550 9450
+F 0 "P?" V 2500 9450 60  0000 C CNN
+F 1 "CONN_20" V 2600 9450 60  0000 C CNN
+F 2 "" H 2550 9450 60  0000 C CNN
+F 3 "" H 2550 9450 60  0000 C CNN
+	1    2550 9450
+	1    0    0    -1
+$EndComp
+$Comp
+L CONN_3X2 P?
+U 1 1 538BDCE4
+P 6700 6350
+F 0 "P?" H 6700 6600 50  0000 C CNN
+F 1 "CONN_3X2" V 6700 6400 40  0000 C CNN
+F 2 "" H 6700 6350 60  0000 C CNN
+F 3 "" H 6700 6350 60  0000 C CNN
+	1    6700 6350
+	1    0    0    -1
+$EndComp
+Entry Wire Line
+	2100 5900 2200 6000
+Entry Wire Line
+	2100 6000 2200 6100
+Entry Wire Line
+	2100 6100 2200 6200
+Entry Wire Line
+	2100 6200 2200 6300
+Entry Wire Line
+	2100 6300 2200 6400
+Entry Wire Line
+	2100 6400 2200 6500
+Entry Wire Line
+	2100 6500 2200 6600
+Entry Wire Line
+	2100 6600 2200 6700
+Entry Wire Line
+	2100 6700 2200 6800
+Entry Wire Line
+	2100 6800 2200 6900
+Entry Wire Line
+	2100 6900 2200 7000
+Entry Wire Line
+	2100 7000 2200 7100
+Entry Wire Line
+	2100 7100 2200 7200
+Entry Wire Line
+	2100 7200 2200 7300
+Entry Wire Line
+	2100 7300 2200 7400
+Entry Wire Line
+	2100 7400 2200 7500
+Entry Wire Line
+	2100 7500 2200 7600
+Entry Wire Line
+	2100 7600 2200 7700
+Entry Wire Line
+	2100 7700 2200 7800
+Entry Wire Line
+	2100 7800 2200 7900
+Entry Wire Line
+	2100 8400 2200 8500
+Entry Wire Line
+	2100 8500 2200 8600
+Entry Wire Line
+	2100 8600 2200 8700
+Entry Wire Line
+	2100 8700 2200 8800
+Entry Wire Line
+	2100 8800 2200 8900
+Entry Wire Line
+	2100 8900 2200 9000
+Entry Wire Line
+	2100 9000 2200 9100
+Entry Wire Line
+	2100 9100 2200 9200
+Entry Wire Line
+	2100 9200 2200 9300
+Entry Wire Line
+	2100 9300 2200 9400
+Entry Wire Line
+	2100 9400 2200 9500
+Entry Wire Line
+	2100 9500 2200 9600
+Entry Wire Line
+	2100 9600 2200 9700
+Entry Wire Line
+	2100 9700 2200 9800
+Entry Wire Line
+	2100 9800 2200 9900
+Entry Wire Line
+	2100 9900 2200 10000
+Entry Wire Line
+	2100 10000 2200 10100
+Entry Wire Line
+	2100 10100 2200 10200
+Entry Wire Line
+	2100 10200 2200 10300
+Entry Wire Line
+	2100 10300 2200 10400
 $EndSCHEMATC
